File: kicad/train-signs.kicad_pcb (KiCad board)
At the start: 2 copper layers, 50.8 x 50.8 mm, 3 parts, among them J1 Conn_02x10_Odd_Even, U1 XIAO ESP32C3

Commit message: Upgraded PCB
Parts:
- added REF**: MountingHole_3.2mm_M3_DIN965_Pad, MountingHole:MountingHole_3.2mm_M3_DIN965_Pad, F.Cu at (54.6, 123.2)
- added REF**: MountingHole_3.2mm_M3_DIN965_Pad, MountingHole:MountingHole_3.2mm_M3_DIN965_Pad, F.Cu at (54.6, 54.6)
- added REF**: MountingHole_3.2mm_M3_DIN965_Pad, MountingHole:MountingHole_3.2mm_M3_DIN965_Pad, F.Cu at (97.5, 54.6)
- moved J1 33.8 mm to (64.8, 89.7), turned to 90 degrees
- moved U1 28.2 mm to (76.3, 113.0)
- moved RV1 12.7 mm to (76.2, 63.5), turned to 90 degrees
Routing:
- net /Contrast: track 56.9 -> 23.5 mm
- net /Board 1 DATA CLK: track 19.5 -> 45.3 mm
- net +5V: track 114.2 -> 88.5 mm
- net /Board 0 DATA CLK: track 19.5 -> 42.5 mm
- net /Board 1 DATA IN: track 19.5 -> 39.9 mm
- net +3V3: track 84.9 -> 104.5 mm
- net /Board 0 CLK: track 38.3 -> 19.1 mm
- net /Board 0 DATA IN: track 19.5 -> 37.4 mm
- net /Board 1 LATCH: track 19.5 -> 34.9 mm
- net /Board 0 LATCH: track 19.5 -> 32.3 mm
- net /Board 1 CLK: track 37.9 -> 25.7 mm
Other:
- board size 50.8 x 50.8 mm -> 50.8 x 76.2 mm
